File: 12V.sch (KiCad schematic (older format))
At the start: 0 parts

Commit message: (Confirmation) BPack Ammeter + Proctection Circuit Edit
Making sure the last commit pushed all edits.
Parts:
- added C?: 10µF, symbol C_Small
- added C? (x2): 0.1µF, symbol C_Small
- added C?: 2.2µF, symbol C_Small
- added C?: C7, symbol C_Small
- added C?: C5, symbol C_Small
- added C?: C_Small, symbol C_Small
- added L?: 1.2µH, symbol L
- added R?: 255kΩ, symbol R_Small
- added R?: R4, symbol R_Small
- added R?: R5, symbol R_Small
- added R?: R2, symbol R_Small
- added R?: R1, symbol R_Small
- added U?: TPS61088, symbol TPS61088
Connections:
- new net: C?.1, U?.1 (VCC)
- new net: C?.2, U?.10 (SS)
- new net: R?.1, R?.1, U?.17 (FB)
- new net: R?.1, U?.18 (COMP)
- new net: R?.1, U?.19 (ILIM)
- new net: R?.1, U?.3 (FSW)
- new net: C?.2, L?.2, R?.2, U?.4 (SW), U?.5 (SW), U?.6 (SW), U?.7 (SW)
- new net: C?.1, U?.8 (BOOT)
- new net: C?.2, R?.2
- new net +9V: C?.1, R?.2, U?.14 (VOUT), U?.15 (VOUT), U?.16 (VOUT)
- new net +BATT: C?.1, C?.2, L?.1, U?.9 (VIN)
- new net GND: C?.1, C?.1, C?.1, C?.2, C?.2, C?.2, R?.2, R?.2, U?.20 (AGND), U?.21 (PGND)
Other:
- note added: "Finish constructing circuit"

Commit message: Changed footprint of TPS61088
Will reconstruct boost converter circuit
Parts:
- removed C?: 10µF, symbol C_Small
- removed C? (x2): 0.1µF, symbol C_Small
- removed C?: 2.2µF, symbol C_Small
- removed C?: C7, symbol C_Small
- removed C?: C5, symbol C_Small
- removed C?: C_Small, symbol C_Small
- removed L?: 1.2µH, symbol L
- removed R?: 255kΩ, symbol R_Small
- removed R?: R4, symbol R_Small
- removed R?: R5, symbol R_Small
- removed R?: R2, symbol R_Small
- removed R?: R1, symbol R_Small
- removed U?: TPS61088, symbol TPS61088
Other:
- note removed: "Finish constructing circuit"
