File: 12V.sch (KiCad schematic (older format))
At the start: 14 parts

Commit message: Ammetre addition
Ammetres added to 3V3 buck converter. Naming convention added for 3V3 1 and 2.
Parts:
- U?: symbol TPS61088 -> TPS61088-RESCUE-eps_v1
Other:
- moved on the sheet: U?
Changed lines of the file:
@@
 EESchema Schematic File Version 2
+LIBS:eps_v1-rescue
 LIBS:power
 LIBS:device
@@
 $EndDescr
 $Comp
-L TPS61088 U?
+L TPS61088-RESCUE-eps_v1 U?
 U 1 1 59E9411F
 P 5150 4700
