File: BATT.sch (KiCad schematic (older format))
At the start: 9 parts

Commit message: Edits to Hierarchical Labels
Added hierarchical labels and changed some in/out directions. Not entirely sure about PV and BP labels.
Changed lines of the file:
@@
 Wire Wire Line
 	6950 2200 6950 2000
-Text HLabel 7100 2000 3    60   Input ~ 0
+Text HLabel 7100 2000 3    60   Output ~ 0
 IPACK
 Text Label 7300 1950 0    60   ~ 0

Commit message: Completed charge controller circuit
Batteries are now on a separate board, and will connect to the EPS
board through header pins. Charge controller circuit was implemented
according to the datasheet.
Parts:
- removed J?: BATTERY, symbol CONN_01X04_MALE
- added J?: -BATT, symbol Conn_02x10_Top_Bottom
- added J?: +BATT, symbol Conn_02x10_Top_Bottom
Connections:
- net labels removed: Original: Batteries 2 and 3 shorted to +PACK
- wire segments 28 -> 32
Other:
- note removed: "Protection for 2 and 4"
- moved on the sheet: R?
Changed lines of the file:
@@
-$EndComp
-$Comp
-L CONN_01X04_MALE J?
-U 1 1 59EA529A
-P 6000 3750
-F 0 "J?" H 6000 4125 50  0000 C CNN
-F 1 "BATTERY" H 6000 3350 50  0000 C CNN
-F 2 "" H 6000 4050 50  0001 C CNN
-F 3 "" H 6000 4050 50  0001 C CNN
-	1    6000 3750
-	0    -1   -1   0
 $EndComp
 $Comp
@@
 L R_Small R?
 U 1 1 59EA52AF
-P 3650 3450
-F 0 "R?" H 3680 3470 50  0000 L CNN
-F 1 "2.2k" H 3680 3410 50  0000 L CNN
-F 2 "" H 3650 3450 50  0001 C CNN
-F 3 "" H 3650 3450 50  0001 C CNN
-	1    3650 3450
-	1    0    0    -1
-$EndComp
-$Comp
-L R_Small R?
-U 1 1 59EA52B6
-P 6500 2650
-F 0 "R?" H 6530 2670 50  0000 L CNN
-F 1 "330" H 6530 2610 50  0000 L CNN
-F 2 "" H 6500 2650 50  0001 C CNN
-F 3 "" H 6500 2650 50  0001 C CNN
-	1    6500 2650
+P 3650 2850
+F 0 "R?" H 3680 2870 50  0000 L CNN
+F 1 "2.2k" H 3680 2810 50  0000 L CNN
+F 2 "" H 3650 2850 50  0001 C CNN
+F 3 "" H 3650 2850 50  0001 C CNN
+	1    3650 2850
 	1    0    0    -1
 $EndComp
@@
 $EndComp
 $Comp
-L -PACK #PWR?
-U 1 1 59EA52C4
-P 4350 3150
-F 0 "#PWR?" H 4350 3000 50  0001 C CNN
-F 1 "-PACK" H 4350 3290 50  0000 C CNN
-F 2 "" H 4350 3150 50  0001 C CNN
-F 3 "" H 4350 3150 50  0001 C CNN
-	1    4350 3150
-	1    0    0    -1
-$EndComp
-$Comp
 L +PACK #PWR?
 U 1 1 59EA52CA
@@
 Text Notes 3850 2450 0    60   ~ 0
 BATTERY AND PROTECTION CIRCUIT
-Wire Wire Line
-	3650 3900 5100 3900
-Connection ~ 4250 3900
-Connection ~ 4350 3900
-Connection ~ 4450 3900
-Connection ~ 4800 3900
-Connection ~ 4900 3900
-Connection ~ 5000 3900
-Wire Wire Line
-	4150 3150 4150 2750
-Wire Wire Line
-	4150 2750 5200 2750
-Wire Wire Line
-	4800 3150 4800 2850
-Wire Wire Line
-	4800 2850 5200 2850
-Wire Wire Line
-	4250 3150 4450 3150
-Connection ~ 4350 3150
-Wire Wire Line
-	4900 3150 5100 3150
-Connection ~ 5000 3150
-Wire Wire Line
-	6100 2750 6500 2750
-Wire Wire Line
-	6500 2750 6500 2850
-Wire Wire Line
-	5000 3150 6500 3150
-Wire Wire Line
-	6500 3150 6500 3050
-Wire Wire Line
-	5700 3450 5700 3350
-Wire Wire Line
-	6300 3350 6300 3450
-Wire Wire Line
-	5700 3350 6300 3350
-Connection ~ 5900 3350
-Wire Wire Line
-	3650 3900 3650 3550
-Connection ~ 4150 3900
-Wire Wire Line
-	3650 3350 3650 2500
-Wire Wire Line
-	3650 2500 6100 2500
-Wire Wire Line
-	6100 2500 6100 2650
-Wire Wire Line
-	5900 3150 5900 3450
-Connection ~ 5900 3150
-Wire Wire Line
-	6100 2850 6100 3150
-Connection ~ 6100 3150
-Text HLabel 6550 2550 1    60   Input ~ 0
+Text HLabel 7050 2550 3    60   Input ~ 0
 +PACK
-Text Notes 5500 4150 0    60   ~ 0
-Protection for 2 and 4
 $Comp
 L INA214 U?
@@
 	0    1    1    0
 $EndComp
-Text Label 5500 4300 0    60   ~ 0
-Original: Batteries 2 and 3 shorted to +PACK
-Wire Wire Line
-	6100 3350 6100 3450
-Connection ~ 6100 3350
 $Comp
 L R_Small R?
@@
 	0    -1   -1   0
 $EndComp
-Wire Wire Line
-	7000 2550 7050 2550
-Wire Wire Line
-	6500 2550 6800 2550
-Wire Wire Line
-	6800 2550 6800 2000
-Wire Wire Line
-	6950 1200 7100 1200
 $Comp
 L +3V3 #PWR?
@@
 	0    1    1    0
 $EndComp
-Wire Wire Line
-	7000 2550 7000 2200
-Wire Wire Line
-	7000 2200 6950 2200
-Wire Wire Line
-	6950 2200 6950 2000
 Text HLabel 7100 2000 3    60   Output ~ 0
 IPACK
 Text Label 7300 1950 0    60   ~ 0
 Output to port expander
+$Comp
+L Conn_02x10_Top_Bottom J?
+U 1 1 5A4805FA
+P 6700 4550
+F 0 "J?" H 6750 5050 50  0000 C CNN
+F 1 "-BATT" H 6750 3950 50  0000 C CNN
+F 2 "" H 6700 4550 50  0001 C CNN
+F 3 "" H 6700 4550 50  0001 C CNN
+	1    6700 4550
+	0    1    1    0
+$EndComp
+$Comp
+L Conn_02x10_Top_Bottom J?
+U 1 1 5A480EC8
+P 6700 3850
+F 0 "J?" H 6750 4350 50  0000 C CNN
+F 1 "+BATT" H 6750 3250 50  0000 C CNN
+F 2 "" H 6700 3850 50  0001 C CNN
+F 3 "" H 6700 3850 50  0001 C CNN
+	1    6700 3850
+	0    1    1    0
+$EndComp
+$Comp
+L GND #PWR?
+U 1 1 5A481828
+P 5750 4350
+F 0 "#PWR?" H 5750 4100 50  0001 C CNN
+F 1 "GND" H 5750 4200 50  0000 C CNN
+F 2 "" H 5750 4350 50  0001 C CNN
+F 3 "" H 5750 4350 50  0001 C CNN
+	1    5750 4350
+	1    0    0    -1
+$EndComp
+$Comp
+L GND #PWR?
+U 1 1 5A481904
+P 6500 3150
+F 0 "#PWR?" H 6500 2900 50  0001 C CNN
+F 1 "GND" H 6500 3000 50  0000 C CNN
+F 2 "" H 6500 3150 50  0001 C CNN
+F 3 "" H 6500 3150 50  0001 C CNN
+	1    6500 3150
+	1    0    0    -1
+$EndComp
+Connection ~ 6200 4350
+Connection ~ 6200 4850
+Wire Wire Line
+	6000 4350 6000 4850
+Connection ~ 6300 4350
+Connection ~ 6400 4350
+Connection ~ 6500 4350
+Connection ~ 6600 4350
+Connection ~ 6700 4350
+Connection ~ 6800 4350
+Connection ~ 6900 4350
+Connection ~ 7000 4350
+Wire Wire Line
+	5750 4350 7100 4350
+Connection ~ 6300 4850
+Connection ~ 6400 4850
+Connection ~ 6500 4850
+Connection ~ 6600 4850
+Connection ~ 6700 4850
+Connection ~ 6800 4850
+Connection ~ 6900 4850
+Connection ~ 7000 4850
+Wire Wire Line
+	6000 4850 7100 4850
+Wire Wire Line
+	6950 2200 6950 2000
+Wire Wire Line
+	7000 2200 6950 2200
+Wire Wire Line
+	7000 2550 7000 2200
+Wire Wire Line
+	6950 1200 7100 1200
+Wire Wire Line
+	6800 2000 6800 3650
+Wire Wire Line
+	6500 2550 6800 2550
+Wire Wire Line
+	7000 2550 7050 2550
+Wire Wire Line
+	6100 3150 6100 2850
+Wire Wire Line
+	6100 2500 6100 2650
+Wire Wire Line
+	3650 2500 6100 2500
+Wire Wire Line
+	6500 3150 6500 3050
+Wire Wire Line
+	6500 2750 6500 2850
+Wire Wire Line
+	6100 2750 6500 2750
+Connection ~ 5000 3150
+Wire Wire Line
+	4900 3150 6100 3150
+Connection ~ 4350 3150
+Wire Wire Line
+	4800 2850 5200 2850
+Wire Wire Line
+	4800 3150 4800 2850
+Wire Wire Line
+	4150 2750 5200 2750
+Wire Wire Line
+	4150 3150 4150 2750
+Connection ~ 5000 3900
+Connection ~ 4900 3900
+Connection ~ 4800 3900
+Connection ~ 4450 3900
+Connection ~ 4350 3900
+Connection ~ 4250 3900
+Connection ~ 6200 3650
+Connection ~ 6200 4150
+Wire Wire Line
+	6000 3650 6000 4150
+Connection ~ 6300 3650
+Connection ~ 6400 3650
+Connection ~ 6500 3650
+Connection ~ 6600 3650
+Connection ~ 6700 3650
+Connection ~ 6800 3650
+Connection ~ 6900 3650
+Connection ~ 7000 3650
+Wire Wire Line
+	6000 3650 7100 3650
+Connection ~ 6300 4150
+Connection ~ 6400 4150
+Connection ~ 6500 4150
+Connection ~ 6600 4150
+Connection ~ 6700 4150
+Connection ~ 6800 4150
+Connection ~ 6900 4150
+Connection ~ 7000 4150
+Wire Wire Line
+	6000 4150 7100 4150
+Wire Wire Line
+	5750 3150 5750 4350
+Connection ~ 6000 4350
+$Comp
+L R_Small R?
+U 1 1 59EA52B6
+P 6500 2650
+F 0 "R?" H 6530 2670 50  0000 L CNN
+F 1 "330" H 6530 2610 50  0000 L CNN
+F 2 "" H 6500 2650 50  0001 C CNN
+F 3 "" H 6500 2650 50  0001 C CNN
+	1    6500 2650
+	1    0    0    -1
+$EndComp
+Connection ~ 6800 2550
+Wire Wire Line
+	3650 2500 3650 2750
+Connection ~ 4250 3150
+Wire Wire Line
+	3650 2950 3650 3050
+Wire Wire Line
+	3650 3050 4450 3050
+Wire Wire Line
+	4450 3050 4450 3150
+Wire Wire Line
+	4350 3150 4350 3050
+Connection ~ 4350 3050
+Wire Wire Line
+	4250 3150 4250 3050
+Connection ~ 4250 3050
+Wire Wire Line
+	4150 3900 5100 3900
+Connection ~ 5750 3150
+Connection ~ 5100 3150
+$Comp
+L -PACK #PWR?
+U 1 1 5A48370F
+P 3650 3050
+F 0 "#PWR?" H 3650 2900 50  0001 C CNN
+F 1 "-PACK" H 3650 3190 50  0000 C CNN
+F 2 "" H 3650 3050 50  0001 C CNN
+F 3 "" H 3650 3050 50  0001 C CNN
+	1    3650 3050
+	-1   0    0    1
+$EndComp
+Text HLabel 3650 3050 0    60   Output ~ 0
+-PACK
 $EndSCHEMATC
