File: _saved_BATT.sch (KiCad schematic (older format))
At the start: 10 parts

Commit message: Created netlist
Still missing deployment and RBL switches
Parts:
- gave numbers to parts that had none: 10
Changed lines of the file:
@@
 $EndDescr
 $Comp
-L bq297xx U?
+L bq297xx U12
 U 1 1 59EA5293
 P 5650 2750
-F 0 "U?" H 5450 2950 60  0000 C CNN
+F 0 "U12" H 5450 2950 60  0000 C CNN
 F 1 "bq297xx" H 5600 2550 60  0000 C CNN
 F 2 "" H 5500 2450 60  0001 C CNN
@@
 $EndComp
 $Comp
-L BSC026NE2LS5 Q?
+L BSC026NE2LS5 Q5
 U 1 1 59EA52A1
 P 4300 3550
-F 0 "Q?" H 4150 3800 60  0000 C CNN
+F 0 "Q5" H 4150 3800 60  0000 C CNN
 F 1 "BSC026NE2LS5" H 4450 3300 60  0000 C CNN
 F 2 "" H 4300 3550 60  0001 C CNN
@@
 $EndComp
 $Comp
-L BSC026NE2LS5 Q?
+L BSC026NE2LS5 Q6
 U 1 1 59EA52A8
 P 4950 3550
-F 0 "Q?" H 4800 3800 60  0000 C CNN
+F 0 "Q6" H 4800 3800 60  0000 C CNN
 F 1 "BSC026NE2LS5" H 5100 3300 60  0000 C CNN
 F 2 "" H 4950 3550 60  0001 C CNN
@@
 $EndComp
 $Comp
-L R_Small R?
+L R_Small R11
 U 1 1 59EA52AF
 P 3650 2850
-F 0 "R?" H 3680 2870 50  0000 L CNN
+F 0 "R11" H 3680 2870 50  0000 L CNN
 F 1 "2.2k" H 3680 2810 50  0000 L CNN
 F 2 "" H 3650 2850 50  0001 C CNN
@@
 $EndComp
 $Comp
-L C_Small C?
+L C_Small C8
 U 1 1 59EA52BD
 P 6500 2950
-F 0 "C?" H 6510 3020 50  0000 L CNN
+F 0 "C8" H 6510 3020 50  0000 L CNN
 F 1 "0.1uF" H 6510 2870 50  0000 L CNN
 F 2 "" H 6500 2950 50  0001 C CNN
@@
 $EndComp
 $Comp
-L +PACK #PWR054
+L +PACK #PWR58
 U 1 1 59EA52CA
 P 7050 2550
-F 0 "#PWR054" H 7050 2400 50  0001 C CNN
+F 0 "#PWR58" H 7050 2400 50  0001 C CNN
 F 1 "+PACK" H 7050 2690 50  0000 C CNN
 F 2 "" H 7050 2550 50  0001 C CNN
@@
 +PACK
 $Comp
-L INA214 U?
+L INA214 U13
 U 1 1 5A10F7B5
 P 6950 1600
-F 0 "U?" H 6950 1300 60  0000 C CNN
+F 0 "U13" H 6950 1300 60  0000 C CNN
 F 1 "INA214" H 6950 1900 60  0000 C CNN
 F 2 "" H 6950 1900 60  0001 C CNN
@@
 $EndComp
 $Comp
-L R_Small R?
+L R_Small R13
 U 1 1 5A112EB5
 P 6900 2550
-F 0 "R?" H 6930 2570 50  0000 L CNN
+F 0 "R13" H 6930 2570 50  0000 L CNN
 F 1 "R_Small" H 6930 2510 50  0000 L CNN
 F 2 "" H 6900 2550 50  0001 C CNN
@@
 $EndComp
 $Comp
-L +3V3 #PWR055
+L +3V3 #PWR59
 U 1 1 5A113C8A
 P 7100 1200
-F 0 "#PWR055" H 7100 1050 50  0001 C CNN
+F 0 "#PWR59" H 7100 1050 50  0001 C CNN
 F 1 "+3V3" H 7100 1340 50  0000 C CNN
 F 2 "" H 7100 1200 50  0001 C CNN
@@
 $EndComp
 $Comp
-L GND #PWR056
+L GND #PWR57
 U 1 1 5A113CE6
 P 6800 1200
-F 0 "#PWR056" H 6800 950 50  0001 C CNN
+F 0 "#PWR57" H 6800 950 50  0001 C CNN
 F 1 "GND" H 6800 1050 50  0000 C CNN
 F 2 "" H 6800 1200 50  0001 C CNN
@@
 Output to port expander
 $Comp
-L Conn_02x10_Top_Bottom J?
+L Conn_02x10_Top_Bottom J6
 U 1 1 5A4805FA
 P 6700 4550
-F 0 "J?" H 6750 5050 50  0000 C CNN
+F 0 "J6" H 6750 5050 50  0000 C CNN
 F 1 "-BATT" H 6750 3950 50  0000 C CNN
 F 2 "" H 6700 4550 50  0001 C CNN
@@
 $EndComp
 $Comp
-L Conn_02x10_Top_Bottom J?
+L Conn_02x10_Top_Bottom J5
 U 1 1 5A480EC8
 P 6700 3850
-F 0 "J?" H 6750 4350 50  0000 C CNN
+F 0 "J5" H 6750 4350 50  0000 C CNN
 F 1 "+BATT" H 6750 3250 50  0000 C CNN
 F 2 "" H 6700 3850 50  0001 C CNN
@@
 $EndComp
 $Comp
-L GND #PWR057
+L GND #PWR55
 U 1 1 5A481828
 P 5750 4350
-F 0 "#PWR057" H 5750 4100 50  0001 C CNN
+F 0 "#PWR55" H 5750 4100 50  0001 C CNN
 F 1 "GND" H 5750 4200 50  0000 C CNN
 F 2 "" H 5750 4350 50  0001 C CNN
@@
 $EndComp
 $Comp
-L GND #PWR058
+L GND #PWR56
 U 1 1 5A481904
 P 6500 3150
-F 0 "#PWR058" H 6500 2900 50  0001 C CNN
+F 0 "#PWR56" H 6500 2900 50  0001 C CNN
 F 1 "GND" H 6500 3000 50  0000 C CNN
 F 2 "" H 6500 3150 50  0001 C CNN
@@
 Connection ~ 6000 4350
 $Comp
-L R_Small R?
+L R_Small R12
 U 1 1 59EA52B6
 P 6500 2650
-F 0 "R?" H 6530 2670 50  0000 L CNN
+F 0 "R12" H 6530 2670 50  0000 L CNN
 F 1 "330" H 6530 2610 50  0000 L CNN
 F 2 "" H 6500 2650 50  0001 C CNN
@@
 Connection ~ 5100 3150
 $Comp
-L -PACK #PWR059
+L -PACK #PWR54
 U 1 1 5A48370F
 P 3650 3050
-F 0 "#PWR059" H 3650 2900 50  0001 C CNN
+F 0 "#PWR54" H 3650 2900 50  0001 C CNN
 F 1 "-PACK" H 3650 3190 50  0000 C CNN
 F 2 "" H 3650 3050 50  0001 C CNN
