File: _saved_PV.sch (KiCad schematic (older format))
At the start: 30 parts

Commit message: Created netlist
Still missing deployment and RBL switches
Parts:
- gave numbers to parts that had none: 30
