File: SWITCH_9V.sch (KiCad schematic (older format))
At the start: 1 part

Commit message: Prototype
Started laying out breakout boards
Parts:
- added R?: R, symbol R
Connections:
- net N_9V: now also R?.1
- new net GND: R?.2
Changed lines of the file:
@@
 Text HLabel 5700 3050 2    60   Output ~ 0
 E_9V
+$Comp
+L GND #PWR?
+U 1 1 5A512F76
+P 4650 2600
+F 0 "#PWR?" H 4650 2350 50  0001 C CNN
+F 1 "GND" H 4650 2450 50  0000 C CNN
+F 2 "" H 4650 2600 50  0001 C CNN
+F 3 "" H 4650 2600 50  0001 C CNN
+	1    4650 2600
+	1    0    0    -1
+$EndComp
+$Comp
+L R R?
+U 1 1 5A512F8D
+P 4650 2450
+F 0 "R?" V 4730 2450 50  0000 C CNN
+F 1 "R" V 4650 2450 50  0000 C CNN
+F 2 "" V 4580 2450 50  0001 C CNN
+F 3 "" H 4650 2450 50  0001 C CNN
+	1    4650 2450
+	1    0    0    -1
+$EndComp
+Connection ~ 4650 2300
 $EndSCHEMATC

Commit message: PCB layout as of 2018-02-07
Parts:
- Q8: renamed from Q?; footprint (none) -> Housings_SON:VSONP-8-1EP_5x6_Pitch1.27mm
- gave numbers to parts that had none: 1
Changed lines of the file:
@@
 $EndDescr
 $Comp
-L +9V #PWR068
+L +9V #PWR084
 U 1 1 5A234B73
 P 2100 1950
-F 0 "#PWR068" H 2100 1800 50  0001 C CNN
+F 0 "#PWR084" H 2100 1800 50  0001 C CNN
 F 1 "+9V" H 2100 2090 50  0000 C CNN
 F 2 "" H 2100 1950 50  0001 C CNN
@@
 $EndComp
 $Comp
-L BSC026NE2LS5 Q?
+L BSC026NE2LS5 Q8
 U 1 1 5A234B8E
 P 3800 2350
-F 0 "Q?" H 3650 2600 60  0000 C CNN
+F 0 "Q8" H 3650 2600 60  0000 C CNN
 F 1 "BSC026NE2LS5" H 3950 2100 60  0000 C CNN
-F 2 "" H 3800 2350 60  0001 C CNN
+F 2 "Housings_SON:VSONP-8-1EP_5x6_Pitch1.27mm" H 3800 2350 60  0001 C CNN
 F 3 "" H 3800 2350 60  0001 C CNN
 	1    3800 2350
@@
 E_9V
 $Comp
-L GND #PWR069
+L GND #PWR085
 U 1 1 5A512F76
 P 4650 2600
-F 0 "#PWR069" H 4650 2350 50  0001 C CNN
+F 0 "#PWR085" H 4650 2350 50  0001 C CNN
 F 1 "GND" H 4650 2450 50  0000 C CNN
 F 2 "" H 4650 2600 50  0001 C CNN
@@
 $EndComp
 $Comp
-L R R?
+L R R22
 U 1 1 5A512F8D
 P 4650 2450
-F 0 "R?" V 4730 2450 50  0000 C CNN
+F 0 "R22" V 4730 2450 50  0000 C CNN
 F 1 "R" V 4650 2450 50  0000 C CNN
 F 2 "" V 4580 2450 50  0001 C CNN
