File: SWITCH_3V3.sch (KiCad schematic (older format))
At the start: 1 part

Commit message: Prototype
Started laying out breakout boards
Parts:
- added R?: R, symbol R
Connections:
- net labels added: GND
- wire segments 7 -> 9
Changed lines of the file:
@@
 Text HLabel 6750 4000 2    60   Output ~ 0
 E_3V3
+$Comp
+L GND #PWR?
+U 1 1 5A5132DF
+P 5800 3550
+F 0 "#PWR?" H 5800 3300 50  0001 C CNN
+F 1 "GND" H 5800 3400 50  0000 C CNN
+F 2 "" H 5800 3550 50  0001 C CNN
+F 3 "" H 5800 3550 50  0001 C CNN
+	1    5800 3550
+	1    0    0    -1
+$EndComp
+$Comp
+L R R?
+U 1 1 5A5132F6
+P 5800 3250
+F 0 "R?" V 5880 3250 50  0000 C CNN
+F 1 "R" V 5800 3250 50  0000 C CNN
+F 2 "" V 5730 3250 50  0001 C CNN
+F 3 "" H 5800 3250 50  0001 C CNN
+	1    5800 3250
+	1    0    0    -1
+$EndComp
+Wire Wire Line
+	5800 3000 5800 3100
+Connection ~ 5800 3000
+Wire Wire Line
+	5800 3400 5800 3550
 $EndSCHEMATC

Commit message: PCB layout as of 2018-02-07
Parts:
- Q7: renamed from Q?; footprint (none) -> Housings_SON:VSONP-8-1EP_5x6_Pitch1.27mm
- gave numbers to parts that had none: 1
Changed lines of the file:
@@
 $EndDescr
 $Comp
-L +3V3 #PWR066
+L +3V3 #PWR082
 U 1 1 5A22FCBF
 P 3150 2550
-F 0 "#PWR066" H 3150 2400 50  0001 C CNN
+F 0 "#PWR082" H 3150 2400 50  0001 C CNN
 F 1 "+3V3" H 3150 2690 50  0000 C CNN
 F 2 "" H 3150 2550 50  0001 C CNN
@@
 	3150 2900 4350 2900
 $Comp
-L BSC026NE2LS5 Q?
+L BSC026NE2LS5 Q7
 U 1 1 5A230963
 P 4700 3050
-F 0 "Q?" H 4550 3300 60  0000 C CNN
+F 0 "Q7" H 4550 3300 60  0000 C CNN
 F 1 "BSC026NE2LS5" H 4850 2800 60  0000 C CNN
-F 2 "" H 4700 3050 60  0001 C CNN
+F 2 "Housings_SON:VSONP-8-1EP_5x6_Pitch1.27mm" H 4700 3050 60  0001 C CNN
 F 3 "" H 4700 3050 60  0001 C CNN
 	1    4700 3050
@@
 E_3V3
 $Comp
-L GND #PWR067
+L GND #PWR083
 U 1 1 5A5132DF
 P 5800 3550
-F 0 "#PWR067" H 5800 3300 50  0001 C CNN
+F 0 "#PWR083" H 5800 3300 50  0001 C CNN
 F 1 "GND" H 5800 3400 50  0000 C CNN
 F 2 "" H 5800 3550 50  0001 C CNN
@@
 $EndComp
 $Comp
-L R R?
+L R R21
 U 1 1 5A5132F6
 P 5800 3250
-F 0 "R?" V 5880 3250 50  0000 C CNN
+F 0 "R21" V 5880 3250 50  0000 C CNN
 F 1 "R" V 5800 3250 50  0000 C CNN
 F 2 "" V 5730 3250 50  0001 C CNN

Commit message: Added REF5025 for 2.5V reference for ADCs
Parts:
- Q7: footprint Housings_SON:VSONP-8-1EP_5x6_Pitch1.27mm -> (none)
Changed lines of the file:
@@
 LIBS:ads7952
 LIBS:tps630250
+LIBS:ref5025
 LIBS:eps_v1-cache
 EELAYER 25 0
@@
 $Descr A4 11693 8268
 encoding utf-8
-Sheet 6 7
+Sheet 4 7
 Title ""
 Date ""
@@
 $EndDescr
 $Comp
-L +3V3 #PWR089
+L +3V3 #PWR099
 U 1 1 5A22FCBF
 P 3150 2550
-F 0 "#PWR089" H 3150 2400 50  0001 C CNN
+F 0 "#PWR099" H 3150 2400 50  0001 C CNN
 F 1 "+3V3" H 3150 2690 50  0000 C CNN
 F 2 "" H 3150 2550 50  0001 C CNN
@@
 F 0 "Q7" H 4550 3300 60  0000 C CNN
 F 1 "BSC026NE2LS5" H 4850 2800 60  0000 C CNN
-F 2 "Housings_SON:VSONP-8-1EP_5x6_Pitch1.27mm" H 4700 3050 60  0001 C CNN
+F 2 "" H 4700 3050 60  0001 C CNN
 F 3 "" H 4700 3050 60  0001 C CNN
 	1    4700 3050
@@
 E_3V3
 $Comp
-L GND #PWR090
+L GND #PWR0100
 U 1 1 5A5132DF
 P 5800 3550
-F 0 "#PWR090" H 5800 3300 50  0001 C CNN
+F 0 "#PWR0100" H 5800 3300 50  0001 C CNN
 F 1 "GND" H 5800 3400 50  0000 C CNN
 F 2 "" H 5800 3550 50  0001 C CNN
