File: SWITCH_5V.sch (KiCad schematic (older format))
At the start: 2 parts, among them Q8 BSC026NE2LS5

Commit message: Added REF5025 for 2.5V reference for ADCs
Parts:
- Q8: footprint Housings_SON:VSONP-8-1EP_5x6_Pitch1.27mm -> (none)
Changed lines of the file:
@@
 LIBS:ads7952
 LIBS:tps630250
+LIBS:ref5025
 LIBS:eps_v1-cache
 EELAYER 25 0
@@
 $Descr A4 11693 8268
 encoding utf-8
-Sheet 7 7
+Sheet 5 7
 Title ""
 Date ""
@@
 $EndDescr
 $Comp
-L +9V #PWR091
+L +9V #PWR0101
 U 1 1 5A234B73
 P 2100 1950
-F 0 "#PWR091" H 2100 1800 50  0001 C CNN
+F 0 "#PWR0101" H 2100 1800 50  0001 C CNN
 F 1 "+9V" H 2100 2090 50  0000 C CNN
 F 2 "" H 2100 1950 50  0001 C CNN
@@
 F 0 "Q8" H 3650 2600 60  0000 C CNN
 F 1 "BSC026NE2LS5" H 3950 2100 60  0000 C CNN
-F 2 "Housings_SON:VSONP-8-1EP_5x6_Pitch1.27mm" H 3800 2350 60  0001 C CNN
+F 2 "" H 3800 2350 60  0001 C CNN
 F 3 "" H 3800 2350 60  0001 C CNN
 	1    3800 2350
@@
 E_9V
 $Comp
-L GND #PWR092
+L GND #PWR0102
 U 1 1 5A512F76
 P 4650 2600
-F 0 "#PWR092" H 4650 2350 50  0001 C CNN
+F 0 "#PWR0102" H 4650 2350 50  0001 C CNN
 F 1 "GND" H 4650 2450 50  0000 C CNN
 F 2 "" H 4650 2600 50  0001 C CNN
