File: Prototype/_autosave-breakout.kicad_pcb (KiCad board)
At the start: 2 copper layers, 8 parts, among them J2 Conn_02x03_Counter_Clockwise, Q1 BSC026NE2LS5, U1 INA214, U2 bq297xx, U3 LM21215, U4 TPS61088, U5 ADA4891-4

Commit message: Test
hello
Routing:
- net Net-(J2-Pad1): track 0.00 -> 22.7 mm, vias 0 -> 2
Changed lines of the file:
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@@
     (thickness 1.6)
     (drawings 0)
-    (tracks 37)
+    (tracks 47)
     (zones 0)
     (modules 8)
@@
     )
   )
+  (segment (start 29.075836 43.805) (end 29.81 43.805) (width 0.25) (layer F.Cu) (net 68))
+  (segment (start 29.81 43.805) (end 29.955 43.95) (width 0.25) (layer F.Cu) (net 68))
+  (segment (start 30.48 40.64) (end 29.075836 42.044164) (width 0.25) (layer B.Cu) (net 68))
+  (segment (start 29.075836 42.044164) (end 29.075836 43.805) (width 0.25) (layer B.Cu) (net 68))
+  (via (at 29.075836 43.805) (size 0.6) (drill 0.4) (layers F.Cu B.Cu) (net 68))
+  (segment (start 31.75 54.61) (end 32.85 54.61) (width 0.25) (layer F.Cu) (net 68))
+  (segment (start 32.85 54.61) (end 35.190018 52.269982) (width 0.25) (layer F.Cu) (net 68))
+  (segment (start 35.190018 52.269982) (end 35.190018 45.350018) (width 0.25) (layer F.Cu) (net 68))
+  (segment (start 35.190018 45.350018) (end 30.48 40.64) (width 0.25) (layer F.Cu) (net 68))
+  (via (at 30.48 40.64) (size 0.6) (drill 0.4) (layers F.Cu B.Cu) (net 68))
   (segment (start 27.94 44.45) (end 27.94 44.325) (width 0.25) (layer F.Cu) (net 69))
   (via (at 27.94 44.325) (size 0.6) (drill 0.4) (layers F.Cu B.Cu) (net 69))
