File: Prototype_Kivanc Aykac/breakout.sch (KiCad schematic (older format))
At the start: 43 parts, among them J1 Conn_01x10_Male, J10 Conn_01x03_Male, J11 Conn_01x03_Male, J12 Conn_01x02_Male, J13 Conn_01x02_Male, J14 Conn_01x02_Male, J15 Conn_01x03_Male, J16 Conn_01x03_Male, J17 Conn_01x03_Male, J18 Conn_01x07_Male, J19 Conn_01x07_Male, J2 Conn_01x03_Male, J20 Conn_01x10_Male, J21 Conn_01x11_Male, J22 Conn_01x10_Male, J23 Conn_01x10_Male, J24 Conn_01x03_Male, J25 Conn_01x03_Male, J26 Conn_01x03_Male, J27 Conn_01x03_Male, J3 Conn_01x10_Male, J4 Conn_01x07_Male, J5 Conn_01x03_Male, J6 Conn_01x10_Male, J7 Conn_01x07_Male, J8 Conn_01x11_Male, J9 Conn_01x03_Male, Q1 BSC026NE2LS5, Q2 BSC026NE2LS5, U1 INA214, U10 bq297xx, U11 INA214, U2 bq297xx, U3 LM21215, U4 TPS61088, U5 ADA4891-4, U6 INA214, U7 ADA4891-4, U8 TPS61088, U9 LM21215

Commit message: breakout changes for myself
Parts:
- added J28, J29: Conn_01x03_Male, Pin_Headers:Pin_Header_Straight_1x03_Pitch2.54mm, symbol Conn_01x03_Male
- added U12: INA214, kicad-libraries:SC70-6, symbol INA214
Connections:
- new net: J28.1 (Pin_1), U12.1 (REF)
- new net: J28.2 (Pin_2), U12.2 (GND)
- new net: J28.3 (Pin_3), U12.3 (V+)
- new net: J29.1 (Pin_1), U12.4 (IN+)
- new net: J29.2 (Pin_2), U12.5 (IN-)
- new net: J29.3 (Pin_3), U12.6 (OUT)
Changed lines of the file:
@@
 	-1   0    0    -1
 $EndComp
+$Comp
+L INA214 U12
+U 1 1 5A95F2A6
+P 10200 3500
+F 0 "U12" H 10200 3200 60  0000 C CNN
+F 1 "INA214" H 10200 3800 60  0000 C CNN
+F 2 "kicad-libraries:SC70-6" H 10200 3800 60  0001 C CNN
+F 3 "" H 10200 3800 60  0001 C CNN
+	1    10200 3500
+	1    0    0    -1
+$EndComp
+$Comp
+L Conn_01x03_Male J28
+U 1 1 5A95F31C
+P 9450 3450
+F 0 "J28" H 9450 3650 50  0000 C CNN
+F 1 "Conn_01x03_Male" H 9450 3250 50  0000 C CNN
+F 2 "Pin_Headers:Pin_Header_Straight_1x03_Pitch2.54mm" H 9450 3450 50  0001 C CNN
+F 3 "" H 9450 3450 50  0001 C CNN
+	1    9450 3450
+	1    0    0    1
+$EndComp
+$Comp
+L Conn_01x03_Male J29
+U 1 1 5A95F470
+P 10950 3450
+F 0 "J29" H 10950 3650 50  0000 C CNN
+F 1 "Conn_01x03_Male" H 10950 3250 50  0000 C CNN
+F 2 "Pin_Headers:Pin_Header_Straight_1x03_Pitch2.54mm" H 10950 3450 50  0001 C CNN
+F 3 "" H 10950 3450 50  0001 C CNN
+	1    10950 3450
+	-1   0    0    1
+$EndComp
 Wire Wire Line
 	1000 6400 1150 6400
@@
 Wire Wire Line
 	9500 4200 9700 4200
+Wire Wire Line
+	9650 3350 9800 3350
+Wire Wire Line
+	9650 3450 9750 3450
+Wire Wire Line
+	9750 3450 9750 3650
+Wire Wire Line
+	9750 3650 9800 3650
+Wire Wire Line
+	9650 3550 9700 3550
+Wire Wire Line
+	9700 3550 9700 3500
+Wire Wire Line
+	9700 3500 9800 3500
+Wire Wire Line
+	10750 3550 10600 3550
+Wire Wire Line
+	10600 3550 10600 3500
+Wire Wire Line
+	10750 3450 10700 3450
+Wire Wire Line
+	10700 3450 10700 3650
+Wire Wire Line
+	10700 3650 10600 3650
+Wire Wire Line
+	10750 3350 10600 3350
 $EndSCHEMATC
