File: Prototype_Kivanc Aykac/breakout.kicad_pcb (KiCad board)
At the start: 2 copper layers, 40 parts, among them J1 Conn_01x10_Male, J10 Conn_01x03_Male, J11 Conn_01x03_Male, J12 Conn_01x02_Male, J13 Conn_01x02_Male, J14 Conn_01x02_Male, J15 Conn_01x03_Male, J16 Conn_01x03_Male, J17 Conn_01x03_Male, J18 Conn_01x07_Male, J19 Conn_01x07_Male, J2 Conn_01x03_Male, J20 Conn_01x10_Male, J21 Conn_01x11_Male, J22 Conn_01x10_Male, J23 Conn_01x10_Male, J24 Conn_01x03_Male, J25 Conn_01x03_Male, J26 Conn_01x03_Male, J27 Conn_01x03_Male, J3 Conn_01x10_Male, J4 Conn_01x07_Male, J5 Conn_01x03_Male, J6 Conn_01x10_Male, J7 Conn_01x07_Male, J8 Conn_01x11_Male, J9 Conn_01x03_Male, Q1 BSC026NE2LS5, Q2 BSC026NE2LS5, U1 INA214, U10 bq297xx, U11 INA214, U2 bq297xx, U3 LM21215, U4 TPS61088, U5 ADA4891-4, U6 INA214, U7 ADA4891-4, U8 TPS61088, U9 LM21215

Commit message: breakout changes for myself
Parts:
- added J28: Conn_01x03_Male, Pin_Headers:Pin_Header_Straight_1x03_Pitch2.54mm, F.Cu at (43.2, 31.8)
- added J29: Conn_01x03_Male, Pin_Headers:Pin_Header_Straight_1x03_Pitch2.54mm, F.Cu at (48.3, 22.9)
- added U12: INA214, kicad-libraries:SC70-6, F.Cu at (45.7, 27.9)
- moved J1 30.0 mm to (110.5, 43.2), turned to 90 degrees
- moved J3 20.1 mm to (133.3, 29.2), turned to 270 degrees
Routing:
- net Net-(J3-Pad1): track 0.00 -> 11.7 mm
- net Net-(J1-Pad10): track 0.00 -> 11.4 mm
- net Net-(J1-Pad1): track 0.00 -> 10.2 mm
- net Net-(J1-Pad9): track 0.00 -> 10.1 mm
- net Net-(J3-Pad2): track 0.00 -> 9.64 mm
- net Net-(J3-Pad10): track 0.00 -> 9.15 mm
- net Net-(J1-Pad8): track 0.00 -> 8.18 mm
- net Net-(J1-Pad2): track 0.00 -> 8.18 mm
- net Net-(J3-Pad3): track 0.00 -> 7.76 mm
- net Net-(J3-Pad9): track 0.00 -> 7.76 mm
- net Net-(J1-Pad3): track 0.00 -> 6.39 mm
- net Net-(J1-Pad7): track 0.00 -> 6.38 mm
- net Net-(J3-Pad8): track 0.00 -> 5.88 mm
- net Net-(J3-Pad4): track 0.00 -> 5.86 mm
- net Net-(J1-Pad4): track 0.00 -> 5.62 mm
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
Commit message: Completed the breakout for myself
Parts:
- moved J9 42.8 mm to (204.5, 115.6), turned to 90 degrees
- moved J11 38.3 mm to (58.4, 57.1), turned to 180 degrees
- moved U2 36.9 mm to (53.3, 54.6)
- moved J18 30.5 mm to (170.2, 158.8), turned to 90 degrees
- moved J19 25.7 mm to (185.4, 143.5), turned to 270 degrees
- moved J15 22.2 mm to (198.1, 35.6), turned to 90 degrees
- moved J20 21.6 mm to (59.7, 139.7), turned to 90 degrees
- moved U7 20.8 mm to (177.8, 151.4)
- moved J10 19.2 mm to (209.6, 105.4), turned to 270 degrees
- moved J24 16.6 mm to (157.5, 101.6)
- moved J25 9.67 mm to (166.4, 106.7), turned to 180 degrees
- moved J21 5.68 mm to (83.8, 125.7)
- moved J22 2.84 mm to (66.0, 101.6)
- moved J23 1.80 mm to (88.9, 86.4)
Routing:
- net Net-(J21-Pad11): track 0.00 -> 14.6 mm
- net Net-(J8-Pad11): track 0.00 -> 14.3 mm
- net Net-(J21-Pad1): track 0.00 -> 14.1 mm
- net Net-(J8-Pad1): track 0.00 -> 14.1 mm
- net Net-(J6-Pad1): track 0.00 -> 13.4 mm
- net Net-(J22-Pad10): track 0.00 -> 12.4 mm
- net Net-(J20-Pad1): track 0.00 -> 12.1 mm
- net Net-(J20-Pad10): track 0.00 -> 12.0 mm
- net Net-(J23-Pad1): track 0.00 -> 11.5 mm
- net Net-(J21-Pad2): track 0.00 -> 10.9 mm
- net Net-(J8-Pad2): track 0.00 -> 10.9 mm
- net Net-(J22-Pad1): track 0.00 -> 10.9 mm
- net Net-(J6-Pad10): track 0.00 -> 10.8 mm
- net Net-(J21-Pad10): track 0.00 -> 10.4 mm
- net Net-(J23-Pad10): track 0.00 -> 10.4 mm
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